File: CircuitBoard/mejiro_siki.kicad_pcb (KiCad board)
At the start: 2 copper layers, 307.5 x 105 mm, 77 parts, among them J1 MJ-4PP-9, J2 MJ-4PP-9, SW1 SW_Push, SW10 SW_Push, SW11 SW_Push, SW12 SW_Push, SW13 SW_Push, SW14 SW_Push, SW15 SW_Push, SW16 SW_Push, SW17 SW_Push, SW18 SW_Push, SW19 SW_Push, SW2 SW_Push, SW20 SW_Push, SW21 SW_Push, SW22 SW_Push, SW23 SW_Push, SW24 SW_Push, SW25 SW_Push, SW26 SW_Push, SW3 SW_Push, SW4 SW_Push, SW5 SW_Push, SW6 SW_Push, SW7 SW_Push, SW8 SW_Push, SW9 SW_Push, U2 xiao-ble-thruhole

Commit message: 基板更新(laptwing対応)
Parts:
- removed REF** (x14): MountingHole_2.2mm_M2, MountingHole:MountingHole_2.2mm_M2
- removed REF** (x5): StampHole2.54, mejiro_footprint:StampHole2.54
- removed the U2 at (81.2, 106.8)
- removed the U2 at (363.2, 106.5)
- added D27: 1N4148W, Diode_SMD:D_SOD-123, F.Cu at (348.3, 136.8)
- added D28: 1N4148W, Diode_SMD:D_SOD-123, F.Cu at (367.3, 136.8)
- added MB1: mousebites 2mm, myfootprint:mousebites_2.5mm, F.Cu at (218.0, 174.5)
- added MB2: mousebites 2mm, myfootprint:mousebites_2.5mm, F.Cu at (218.0, 149.0)
- added MB3: mousebites 2mm, myfootprint:mousebites_2.5mm, F.Cu at (218.0, 123.5)
- added SP1: MountingHole_6.4mm_M6, MountingHole:MountingHole_6.4mm_M6, F.Cu at (250.9, 147.2)
- added SP10: MountingHole_6.4mm_M6, MountingHole:MountingHole_6.4mm_M6, F.Cu at (207.2, 190.2)
- added SP2: MountingHole_6.4mm_M6, MountingHole:MountingHole_6.4mm_M6, F.Cu at (227.9, 190.2)
- added SP3: MountingHole_6.4mm_M6, MountingHole:MountingHole_6.4mm_M6, F.Cu at (309.9, 147.2)
- added SP4: MountingHole_6.4mm_M6, MountingHole:MountingHole_6.4mm_M6, F.Cu at (371.9, 147.2)
- added SP5: MountingHole_6.4mm_M6, MountingHole:MountingHole_6.4mm_M6, F.Cu at (371.9, 190.2)
- added SP6: MountingHole_6.4mm_M6, MountingHole:MountingHole_6.4mm_M6, F.Cu at (63.2, 190.2)
- added SP7: MountingHole_6.4mm_M6, MountingHole:MountingHole_6.4mm_M6, F.Cu at (86.2, 147.2)
- added SP8: MountingHole_6.4mm_M6, MountingHole:MountingHole_6.4mm_M6, F.Cu at (145.2, 147.2)
- added SP9: MountingHole_6.4mm_M6, MountingHole:MountingHole_6.4mm_M6, F.Cu at (207.2, 147.2)
- added SW27: SW_Push, BrownSugar_KBD:CherryMX_Hotswap_via_1U, F.Cu at (348.3, 129.8)
- added SW28: SW_Push, BrownSugar_KBD:CherryMX_Hotswap_via_1U, F.Cu at (367.3, 129.8)
- added U1: XIAO-RP2040-SMD, XIAO_PCB:XIAO-RP2040-SMD, B.Cu at (197.5, 109.9)
- added U2: XIAO-RP2040-SMD, XIAO_PCB:XIAO-RP2040-SMD, B.Cu at (236.0, 109.9)
- D1, D10, D11, D12, D13, D14, D15, D16, D17, D18, D19, D2, D20, D21, D22, D23, D24, D25, D26, D3, D4, D5, D6, D7, D8, D9: moved to F.Cu
- RSW1: footprint mejiro_footprint:SKHLLCA010 -> myfootprint:SKHLLCA010; moved to B.Cu
- RSW2: footprint mejiro_footprint:SKHLLCA010 -> myfootprint:SKHLLCA010
- SW1, SW10, SW11, SW12, SW13, SW14, SW15, SW16, SW17, SW18, SW19, SW2, SW20, SW21, SW22, SW23, SW24, SW25, SW26, SW3, SW4, SW5, SW6, SW7, SW8, SW9: footprint keyswitches:Kailh_socket_MX -> BrownSugar_KBD:CherryMX_Hotswap_via_1U
- moved D1 213.5 mm to (66.0, 127.0), turned to 180 degrees
- moved D14 210.8 mm to (367.3, 117.8), turned to 0 degrees
- moved D2 200.5 mm to (85.2, 127.2), turned to 180 degrees
- moved D15 198.5 mm to (348.3, 117.8), turned to 0 degrees
- moved RSW1 195.6 mm to (177.2, 103.6), turned to 180 degrees
- moved D4 187.9 mm to (103.9, 136.8), turned to 180 degrees
- moved D3 187.7 mm to (104.7, 117.8), turned to 180 degrees
- moved D16 186.3 mm to (329.3, 117.8), turned to 0 degrees
- moved D17 185.6 mm to (329.3, 136.8), turned to 0 degrees
- moved RSW2 185.1 mm to (256.3, 103.5), turned to 180 degrees
- moved SW12 181.9 mm to (161.2, 186.8)
- moved SW11 181.6 mm to (170.8, 167.8)
- moved SW13 181.4 mm to (180.2, 186.8)
- moved SW8 178.6 mm to (142.2, 129.8)
- moved SW7 178.6 mm to (142.2, 110.9)
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Routing:
- net /COL1_L: track 100.8 -> 195.4 mm, vias 0 -> 1
- net /ROW1_R: track 104.4 -> 182.7 mm, vias 2 -> 1
- net Net-(D2-A): track 102.6 -> 24.7 mm
- net /COL3_R: track 237.4 -> 162.4 mm
- net /COL2_L: track 106.9 -> 178.7 mm, vias 0 -> 1
- net /COL5_R: track 142.6 -> 84.6 mm
- net /RST_L: track 86.2 -> 30.6 mm
- net /ROW2_L: track 103.0 -> 151.8 mm, vias 0 -> 1
- net /COL5_L: track 87.2 -> 136.1 mm, vias 2 -> 1
- net Net-(D26-A): track 63.5 -> 17.0 mm
- net /COL4_L: track 159.1 -> 202.2 mm, vias 2 -> 1
- net /ROW0_L: track 118.9 -> 161.5 mm, vias 0 -> 1
- net /COL4_R: track 189.6 -> 147.3 mm
- net Net-(D25-A): track 59.5 -> 19.1 mm
- net /ROW0_R: track 127.6 -> 167.7 mm, vias 5 -> 1
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- added copper zone on B.Cu, net /GND_L
- added copper zone on F.Cu, net /GND_L
- added copper zone on B.Cu, net /GND_R
- added copper zone on F.Cu, net /GND_R
- added copper zone on F.Cu, net /VCC_R
Other:
- board size 307.5 x 105 mm -> 327 x 102.2 mm
